Commit message: fix

File: src/orbibot_description/urdf/orbibot.urdf.xacro (robot description, xacro)
@@ -12,5 +12,5 @@
   <xacro:property name="base_width" value="0.25"/>
   <xacro:property name="base_height" value="0.10"/>
-  <xacro:property name="base_mass" value="8.5"/>
+  <xacro:property name="base_mass" value="6.0"/>
   <!-- Sensor positions -->
   <xacro:property name="lidar_height" value="0.0"/>

Commit message: debugging

File: src/orbibot_description/urdf/orbibot.urdf.xacro (robot description, xacro)
@@ -101,5 +101,5 @@
     <parent link="base_link"/>
     <child link="lidar_link"/>
-    <origin xyz="0.0 0.0 ${lidar_height}" rpy="${PI/2} 0 ${PI}"/>
+    <origin xyz="0.0 0.0 ${lidar_height}" rpy="0 0 0"/>
   </joint>
   <link name="lidar_link">

Commit message: refactor

File: src/orbibot_description/urdf/orbibot.urdf.xacro (robot description, xacro)
@@ -14,5 +14,5 @@
   <xacro:property name="base_mass" value="6.0"/>
   <!-- Sensor positions -->
-  <xacro:property name="lidar_height" value="0.0"/>
+  <xacro:property name="lidar_height" value="0.06"/>
   <xacro:property name="camera_height" value="0.02"/>
   <!-- Inertia macros -->

Commit message: re-factor

File: src/orbibot_description/urdf/orbibot.urdf.xacro (robot description, xacro)
@@ -14,5 +14,5 @@
   <xacro:property name="base_mass" value="6.0"/>
   <!-- Sensor positions -->
-  <xacro:property name="lidar_height" value="0.06"/>
+  <xacro:property name="lidar_height" value="0.18"/>
   <xacro:property name="camera_height" value="0.02"/>
   <!-- Inertia macros -->
@@ -107,5 +107,5 @@
       <origin xyz="-0.03 0 -0.1" rpy="0 0 0"/>
       <geometry>
-        <mesh filename="package://orbibot_description/meshes/RPLider-A1.stl" scale="0.001 0.001 0.001"/>
+        <mesh filename="package://orbibot_description/meshes/RPLidar-A1.stl" scale="0.001 0.001 0.001"/>
       </geometry>
       <material name="lidar_material">

Commit message: fix bug

File: src/orbibot_description/urdf/orbibot.urdf.xacro (robot description, xacro)
@@ -129,5 +129,5 @@
     <parent link="base_link"/>
     <child link="camera_link"/>
-    <origin xyz="${base_length/2} 0.0 ${camera_height}" rpy="0 0 ${PI/2}"/>
+    <origin xyz="${base_length/2} 0.0 ${camera_height}" rpy="0 0 0"/>
   </joint>
   <link name="camera_link">
@@ -135,5 +135,5 @@
       <origin xyz="0 0 0" rpy="0 0 0"/>
       <geometry>
-        <box size="0.09 0.025 0.025"/>
+        <box size="0.025 0.09 0.025"/>
       </geometry>
       <material name="camera_material">
@@ -144,5 +144,5 @@
       <origin xyz="0 0 0" rpy="0 0 0"/>
       <geometry>
-        <box size="0.09 0.025 0.025"/>
+        <box size="0.025 0.09 0.025"/>
       </geometry>
     </collision>
@@ -150,5 +150,5 @@
       <origin xyz="0 0 0" rpy="0 0 0"/>
       <mass value="0.072"/>
-      <xacro:box_inertia m="0.072" x="0.09" y="0.025" z="0.025"/>
+      <xacro:box_inertia m="0.072" x="0.025" y="0.09" z="0.025"/>
     </inertial>
   </link>
